File: hdw/Ultimate_Counter/Clock_Output.sch (KiCad schematic (older format))
At the start: 7 parts

Commit message: Started on schematic
Parts:
- removed J?: CLK_OUT, Socket_Strips:Socket_Strip_Angled_1x02_Pitch2.54mm, symbol Connector_Generic:Conn_01x02
- removed R?: 100, Resistors_SMD:R_0603, symbol Custom_Library:R_Custom
- added D? (x2): 3.3V, Diodes_SMD:D_SOD-323, symbol Device:D_TVS_ALT
- added J?: Signal_Output, symbol Connector_Generic:Conn_01x04
Connections:
- net GND: now also D?.2 (A2), D?.2 (A2), J?.4 (Pin_4)
- net at D?.1 (A1), R?.2, R?.2: now also J?.1 (Pin_1)
- net Stage10_Clock_Out renamed Stage04_Q11
- new net Count_Reset: D?.1 (A1), J?.2 (Pin_2)
- new net LED_Enable: D?.1 (A1), J?.3 (Pin_3)
Other:
- moved on the sheet: C?, D?, R?, U?
