File: hdw/Ultimate_Counter/Oscillator.sch (KiCad schematic (older format))
At the start: 12 parts

Commit message: Lots of changes:
Parts:
- removed C? (x2): 0.1uF, Capacitors_SMD:C_0603, symbol Custom_Library:C_Custom
- removed R? (x4): 10k, Resistors_SMD:R_0603, symbol Custom_Library:R_Custom
- removed U?: CD4024, Housings_SSOP:TSSOP-14_4.4x5mm_Pitch0.65mm, symbol 74xx:74HC4024
- removed U?: CD4040, Custom Footprints Library:DHVQFN16-1ep_3p5x2p5mm, symbol 4xxx:4040
- removed X?: ECS-327KE, Custom Footprints Library:ECS-327KE, symbol Custom_Library:ECS-327KE
- added C?: 0.1uF, Capacitors_SMD:C_0603, symbol Custom_Library:C_Custom
- added R?: 10k, Resistors_SMD:R_0603, symbol Custom_Library:R_Custom
- added R?: 10, Resistors_SMD:R_0603, symbol Custom_Library:R_Custom
- added U?: MAX7375AXR425, Package_TO_SOT_SMD:SOT-323_SC-70, symbol Oscillator:MAX7375AXR425
- added U?: 74LVC1G32, TO_SOT_Packages_SMD:SOT-353_SC-70-5, symbol Custom_Library:74LVC1G32_Power
Connections:
- net +3V3: now also C?.1, U?.1 (V+), U?.5 (VCC)
- net GND: now also C?.2, R?.2, U?.3 (GND), U?.3 (GND)
- new net: R?.1, R?.2, U?.2 (CLOCK)
- new net External_Clock: U?.1
- new net FAST_OSC: R?.1, U?.2
- new net Stage01_Clock_In: U?.4
- no-connect marks 15 -> 0
Other:
- moved on the sheet: C?
