File: hdw/Ultimate_Counter/POS12_Power_Input.sch (KiCad schematic (older format))
At the start: 19 parts

Commit message: Started on schematic
Parts:
- removed C?: 10nF, Capacitors_SMD:C_0603, symbol Custom_Library:C_Custom
- removed N?: +12V 1A Power Supply, symbol Mechanical:Housing
- removed R? (x2): 10k, Resistors_SMD:R_0603, symbol Custom_Library:R_Custom
- removed R?: 6.04k, Resistors_SMD:R_0603, symbol Custom_Library:R_Custom
- removed R?: 16.5k, Resistors_SMD:R_0603, symbol Custom_Library:R_Custom
- removed R?: 1.15k, Resistors_SMD:R_0603, symbol Custom_Library:R_Custom
- removed R?: 51.1k, Resistors_SMD:R_0603, symbol Custom_Library:R_Custom
- removed R?: 5.11k, Resistors_SMD:R_0603, symbol Custom_Library:R_Custom
- removed TP? (x2): TP_Pad, Custom Footprints Library:Test_Point, symbol Custom_Library:TP_Pad
- removed TP?: TP, Pin_Headers:Pin_Header_Angled_1x01_Pitch2.54mm, symbol Custom_Library:TP
- removed U?: TPS26600RHFT, Housings_DFN_QFN:QFN-24-1EP_4x5mm_Pitch0.5mm, symbol Custom_Library:TPS26600RHFT
- added C?: 0.1uF, Capacitors_SMD:C_0603, symbol Custom_Library:C_Custom
- added N?: +12V 1A Power Supply, symbol Mechanical:Housing
- added Q? (x2): IPC100N04S51R7ATMA1, TO_SOT_Packages_SMD:TDSON-8-1, symbol Custom_Library:IPC100N04S51R7ATMA1
- added R?: 6.04M, Resistors_SMD:R_0603, symbol Custom_Library:R_Custom
- added R?: 86.6k, Resistors_SMD:R_0603, symbol Custom_Library:R_Custom
- added R?: 243k, Resistors_SMD:R_0603, symbol Custom_Library:R_Custom
- added R?: 100k, Resistors_SMD:R_0603, symbol Custom_Library:R_Custom
- added R? (x2): 10, Resistors_SMD:R_0603, symbol Custom_Library:R_Custom
- added R?: 5.1k, Resistors_SMD:R_0603, symbol Custom_Library:R_Custom
- added R?: 13.7k, Resistors_SMD:R_0603, symbol Custom_Library:R_Custom
- added R?: 5.23k, Resistors_SMD:R_0603, symbol Custom_Library:R_Custom
- added TP?: TP, Pin_Headers:Pin_Header_Angled_1x01_Pitch2.54mm, symbol Custom_Library:TP
- added TP? (x2): TP, Custom Footprints Library:Test_Point, symbol Custom_Library:TP
- added U?: LTC4365DDB, Housings_DFN_QFN:DFN-8-1EP_2x3mm_Pitch0.5mm, symbol Custom_Library:LTC4365DDB
Connections:
- net +12V: now also Q?.5 (D), R?.1, TP?.1 (TP), U?.6 (Vout)
- net +12Vin: now also Q?.5 (D), R?.1, R?.1, TP?.1 (TP), U?.4 (Vin)
- net GND: now also C?.2, R?.2, R?.2, TP?.1 (TP), U?.1 (GND), U?.9 (GND)
- net POS12_PGOOD: now also R?.1, R?.2, U?.7 (~FAULT)
- new net: R?.1, R?.2, U?.3 (UV)
- new net: R?.1, R?.2, U?.2 (OV)
- new net: R?.2, U?.8 (~SHDN)
- new net: R?.1, R?.1, R?.2, U?.5 (GATE)
- new net: Q?.4 (G), R?.2
- new net: Q?.4 (G), R?.1
- new net: C?.1, R?.2
- new net: Q?.1 (S), Q?.1 (S), Q?.2 (S), Q?.2 (S), Q?.3 (S), Q?.3 (S)
- no-connect marks 1 -> 0
Other:
- note added: "02. +12V Input"
- note added: "UVLO threshold set to 10V\nOVLO threshold set to 14V"
- note removed: "UVLO threshold set to 10.8V\nOVLO threshold set to 13.2V\n\nMODE set to Circuit Breaker with Auto-Retry"
- moved on the sheet: C?, D?, J?
