File: hdw/Ultimate_Counter/Pushbuttons.sch (KiCad schematic (older format))
At the start: 41 parts

Commit message: Started on schematic
Parts:
- removed C? (x2): 10nF, Capacitors_SMD:C_0603, symbol Custom_Library:C_Custom
- removed C? (x7): 0.1uF, Capacitors_SMD:C_0603, symbol Custom_Library:C_Custom
- removed C? (x2): 10uF, Capacitors_SMD:C_0603, symbol Custom_Library:C_Custom
- removed R? (x2): 499, Resistors_SMD:R_0603, symbol Custom_Library:R_Custom
- removed R? (x6): 10k, Resistors_SMD:R_0603, symbol Custom_Library:R_Custom
- removed SW? (x2): Cap_Touch, Custom Footprints Library:Capacitive_Touch_Pad, symbol Custom_Library:Cap_Touch
- removed U? (x2): AT42QT1010-TSHR, TO_SOT_Packages_SMD:SOT-23-6, symbol Sensor_Touch:AT42QT1010-TSHR
- removed U?: 74LVC1G80, TO_SOT_Packages_SMD:SOT-353_SC-70-5, symbol Custom_Library:74LVC1G80_Power
- removed U? (x2): TLV71330PDBV, Package_TO_SOT_SMD:SOT-23-5, symbol Regulator_Linear:TLV71330PDBV
- removed U? (x2): 74LVC1G17, TO_SOT_Packages_SMD:SOT-353_SC-70-5, symbol Custom_Library:74LVC1G17_Power

Commit message: Lots of changes:
Parts:
- added C?: 10nF, Capacitors_SMD:C_0603, symbol Custom_Library:C_Custom
- added C? (x3): 0.1uF, Capacitors_SMD:C_0603, symbol Custom_Library:C_Custom
- added C?: 10uF, Capacitors_SMD:C_0603, symbol Custom_Library:C_Custom
- added R?: 499, Resistors_SMD:R_0603, symbol Custom_Library:R_Custom
- added R?: 1M, Resistors_SMD:R_0603, symbol Custom_Library:R_Custom
- added R? (x3): 10k, Resistors_SMD:R_0603, symbol Custom_Library:R_Custom
- added SW?: Cap_Touch, Custom Footprints Library:Capacitive_Touch_Pad, symbol Custom_Library:Cap_Touch
- added U?: TLV71330PDBV, Package_TO_SOT_SMD:SOT-23-5, symbol Regulator_Linear:TLV71330PDBV
- added U?: AT42QT1012-T, Package_TO_SOT_SMD:SOT-23-6, symbol Sensor_Touch:AT42QT1012-T
- added U?: 74LVC1G17, TO_SOT_Packages_SMD:SOT-353_SC-70-5, symbol Custom_Library:74LVC1G17_Power
Connections:
- net +3V3: now also C?.1, C?.1, U?.1 (IN), U?.3 (EN), U?.5 (VCC)
- net GND: now also C?.2, C?.2, C?.2, C?.2, R?.2, R?.2, R?.2, U?.2 (GND), U?.2 (VSS), U?.3 (GND), U?.6 (TIME)
- new net: C?.1, R?.1, U?.4 (SNS)
- new net: C?.2, R?.2, U?.3 (SNSK)
- new net: R?.1, SW?.1 (TP)
- new net: C?.1, U?.5 (OUT), U?.5 (VDD)
- new net: R?.1, R?.2, U?.1 (OUT)
- new net: C?.1, R?.1, U?.2
- new net LED_Enable: R?.1, U?.4
Other:
- moved on the sheet: C?, R?, SW?, U?
